File: docs/Kicad Files/Amplifier/Amplifier, REV-A/Dorr_Amp_REV-.kicad_pcb (KiCad board)
At the start: 2 copper layers, 163.8 x 76.2 mm, 48 parts, among them J1 Speaker Terminals, J2 Input Terminals, J3 Power Input, Q1 2N3904, Q10 QD44H8G, Q2 QD45H8G, Q3 2N3904, Q4 2N3906, Q5 QD44H8G, Q6 2N3904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

Commit message: Amp Board Update
Updated the power transistor pins in the schematic to reflect datasheets. Minor changes to component placement.
Parts:
- Q10, Q2: footprint Package_TO_SOT_THT:TO-218-3_Vertical -> Package_TO_SOT_THT:TO-220-3_Vertical
- moved R7 16.7 mm to (57.5, 120.9)
- moved C7 12.4 mm to (162.7, 100.4)
- moved R8 10.7 mm to (67.3, 128.7)
- moved J1 10.2 mm to (181.0, 98.4)
- moved R16 6.14 mm to (129.8, 65.3), turned to -90 degrees
- moved Q2 6.01 mm to (144.9, 95.5), turned to -90 degrees
- moved C1 5.74 mm to (155.3, 100.6)
- moved H4 5.55 mm to (187.3, 134.8)
- moved H2 5.46 mm to (187.4, 66.3)
- moved C8 5.41 mm to (166.6, 81.1)
- moved H3 4.84 mm to (42.0, 134.8)
- moved H1 4.61 mm to (42.3, 66.7)
- moved C4 3.94 mm to (114.7, 132.0), turned to -90 degrees
- moved Q9 3.93 mm to (146.8, 114.4), turned to 90 degrees
- moved Q7 2.66 mm to (114.6, 94.9), turned to -90 degrees
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Connections:
- Q10 pad 1: GND -> Net-(Q10-B)
- Q10 pad 2: Net-(Q10-B) -> Net-(Q10-C)
- Q10 pad 3: Net-(Q10-C) -> GND
- Q2 pad 1: /18V -> Net-(Q2-B)
- Q2 pad 2: Net-(Q2-B) -> Net-(Q2-C)
- Q2 pad 3: Net-(Q2-C) -> /18V
- Q5 pad 1: GND -> Net-(Q4-C)
- Q5 pad 2: Net-(Q4-C) -> Net-(Q4-E)
- Q5 pad 3: Net-(Q4-E) -> GND
- Q9 pad 1: /18V -> Net-(Q1-C)
- Q9 pad 2: Net-(Q1-C) -> Net-(Q1-E)
- Q9 pad 3: Net-(Q1-E) -> /18V
Routing:
- net /18V: track 267.8 -> 104.7 mm
- net GND: track 80.4 -> 1.51 mm, vias 53 -> 0
- net Net-(J1-Pin_2): track 105.4 -> 94.9 mm
- net Net-(C8-Pad1): track 82.9 -> 76.5 mm
- net Net-(J1-Pin_1): track 24.6 -> 20.1 mm
- net Net-(D1-K): track 71.8 -> 67.9 mm
- net Net-(Q10-C): track 41.1 -> 37.2 mm
- net Net-(D3-K): track 62.8 -> 60.1 mm
- net Net-(D4-K): track 37.6 -> 39.9 mm
- net Net-(Q1-C): track 33.0 -> 35.0 mm
- net Net-(Q1-E): track 33.0 -> 34.7 mm
- net Net-(Q2-C): track 33.7 -> 35.2 mm
- net Net-(Q4-C): track 39.9 -> 38.4 mm
- net Net-(Q10-B): track 41.3 -> 42.8 mm
- net Net-(D2-K): track 39.4 -> 40.6 mm
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Other:
- board size 163.8 x 76.2 mm -> 152.7 x 76.2 mm
