File: docs/Kicad Files/Amplifier/Amplifier, REV-/Dorr_Amp_REV-.kicad_sch (KiCad schematic)
At the start: 48 parts, among them J1 Speaker Terminals, J2 Input Terminals, J3 Power Input, Q1 2N3904, Q10 QD44H8G, Q2 QD45H8G, Q3 2N3904, Q4 2N3906, Q5 QD44H8G, Q6 2N3904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

Commit message: Fixed all footprints
All footprints should be good. Need to double check the capacitor lead spacing with those in the lab.
Parts:
- C3, C5: footprint Capacitor_THT:CP_Radial_D4.0mm_P1.50mm -> Capacitor_THT:C_Disc_D4.3mm_W1.9mm_P5.00mm
- C4, C6: footprint Capacitor_THT:CP_Radial_D4.0mm_P1.50mm -> Capacitor_THT:C_Disc_D3.0mm_W1.6mm_P2.50mm
- C8: footprint Capacitor_THT:CP_Radial_D12.5mm_P7.50mm -> Capacitor_THT:CP_Radial_D12.5mm_P5.00mm
- H1, H2, H3, H4: footprint MountingHole:MountingHole_2.7mm_M2.5_DIN965_Pad -> MountingHole:MountingHole_3.5mm_Pad
- J1: value Speaker Terminals -> Speaker; footprint Connector_Wire:SolderWire-2.5sqmm_1x02_P7.2mm_D2.4mm_OD3.6mm -> Z_Custom_Footprints:CONN_1935776_PXC
- J2, J3: footprint Connector_Wire:SolderWire-2.5sqmm_1x02_P7.2mm_D2.4mm_OD3.6mm -> Z_Custom_Footprints:CONN_1935776_PXC
- R1, R10, R12, R13, R14, R15, R16, R17, R18, R2, R3, R4, R5, R6, R8, R9: footprint Resistor_THT:R_Axial_DIN0204_L3.6mm_D1.6mm_P5.08mm_Horizontal -> Resistor_THT:R_Axial_DIN0207_L6.3mm_D2.5mm_P10.16mm_Horizontal
- R11, R7: footprint Potentiometer_THT:Potentiometer_ACP_CA9-V10_Vertical -> Z_Custom_Footprints:POT_3362P
- TP1, TP2: footprint TestPoint:TestPoint_Loop_D2.50mm_Drill1.0mm -> TestPoint:TestPoint_Plated_Hole_D2.0mm
Changed lines of the file:
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@@
 			)
 		)
-		(property "Footprint" "Resistor_THT:R_Axial_DIN0204_L3.6mm_D1.6mm_P5.08mm_Horizontal"
+		(property "Footprint" "Resistor_THT:R_Axial_DIN0207_L6.3mm_D2.5mm_P10.16mm_Horizontal"
 			(at 165.862 55.88 90)
 			(effects
@@
 			)
 		)
-		(property "Footprint" "Resistor_THT:R_Axial_DIN0204_L3.6mm_D1.6mm_P5.08mm_Horizontal"
+		(property "Footprint" "Resistor_THT:R_Axial_DIN0207_L6.3mm_D2.5mm_P10.16mm_Horizontal"
 			(at 140.97 64.008 90)
 			(effects
@@
 			)
 		)
-		(property "Footprint" "Resistor_THT:R_Axial_DIN0204_L3.6mm_D1.6mm_P5.08mm_Horizontal"
+		(property "Footprint" "Resistor_THT:R_Axial_DIN0207_L6.3mm_D2.5mm_P10.16mm_Horizontal"
 			(at 142.24 87.122 90)
 			(effects
@@
 			)
 		)
-		(property "Footprint" "Resistor_THT:R_Axial_DIN0204_L3.6mm_D1.6mm_P5.08mm_Horizontal"
+		(property "Footprint" "Resistor_THT:R_Axial_DIN0207_L6.3mm_D2.5mm_P10.16mm_Horizontal"
 			(at 110.49 103.632 90)
 			(effects
@@
 			)
 		)
-		(property "Footprint" "Capacitor_THT:CP_Radial_D12.5mm_P7.50mm"
+		(property "Footprint" "Capacitor_THT:CP_Radial_D12.5mm_P5.00mm"
 			(at 199.39 63.1952 0)
 			(effects
@@
 			)
 		)
-		(property "Footprint" "Resistor_THT:R_Axial_DIN0204_L3.6mm_D1.6mm_P5.08mm_Horizontal"
+		(property "Footprint" "Resistor_THT:R_Axial_DIN0207_L6.3mm_D2.5mm_P10.16mm_Horizontal"
 			(at 165.862 111.76 90)
 			(effects
@@
 			)
 		)
-		(property "Footprint" "Capacitor_THT:CP_Radial_D4.0mm_P1.50mm"
+		(property "Footprint" "Capacitor_THT:C_Disc_D4.3mm_W1.9mm_P5.00mm"
 			(at 97.79 104.4448 0)
 			(effects
@@
 			)
 		)
-		(property "Footprint" "TestPoint:TestPoint_Loop_D2.50mm_Drill1.0mm"
+		(property "Footprint" "TestPoint:TestPoint_Plated_Hole_D2.0mm"
 			(at 184.15 62.23 0)
 			(effects
@@
 			)
 		)
-		(property "Footprint" "TestPoint:TestPoint_Loop_D2.50mm_Drill1.0mm"
+		(property "Footprint" "TestPoint:TestPoint_Plated_Hole_D2.0mm"
 			(at 184.15 105.41 0)
 			(effects
@@
 			)
 		)
-		(property "Footprint" "Potentiometer_THT:Potentiometer_ACP_CA9-V10_Vertical"
+		(property "Footprint" "Z_Custom_Footprints:POT_3362P"
 			(at 110.49 126.238 90)
 			(effects
@@
 			)
 		)
-		(property "Footprint" "Resistor_THT:R_Axial_DIN0204_L3.6mm_D1.6mm_P5.08mm_Horizontal"
+		(property "Footprint" "Resistor_THT:R_Axial_DIN0207_L6.3mm_D2.5mm_P10.16mm_Horizontal"
 			(at 125.222 80.01 90)
 			(effects
@@
 			)
 		)
-		(property "Footprint" "Resistor_THT:R_Axial_DIN0204_L3.6mm_D1.6mm_P5.08mm_Horizontal"
+		(property "Footprint" "Resistor_THT:R_Axial_DIN0207_L6.3mm_D2.5mm_P10.16mm_Horizontal"
 			(at 110.49 64.008 90)
 			(effects
@@
 			)
 		)
-		(property "Footprint" "Resistor_THT:R_Axial_DIN0204_L3.6mm_D1.6mm_P5.08mm_Horizontal"
+		(property "Footprint" "Resistor_THT:R_Axial_DIN0207_L6.3mm_D2.5mm_P10.16mm_Horizontal"
 			(at 155.702 35.56 90)
 			(effects
@@
 			)
 		)
-		(property "Footprint" "Connector_Wire:SolderWire-2.5sqmm_1x02_P7.2mm_D2.4mm_OD3.6mm"
+		(property "Footprint" "Z_Custom_Footprints:CONN_1935776_PXC"
 			(at 83.82 83.82 0)
 			(effects
@@
 			)
 		)
-		(property "Footprint" "Resistor_THT:R_Axial_DIN0204_L3.6mm_D1.6mm_P5.08mm_Horizontal"
+		(property "Footprint" "Resistor_THT:R_Axial_DIN0207_L6.3mm_D2.5mm_P10.16mm_Horizontal"
 			(at 140.97 103.632 90)
 			(effects
@@
 			)
 		)
-		(property "Footprint" "Connector_Wire:SolderWire-2.5sqmm_1x02_P7.2mm_D2.4mm_OD3.6mm"
+		(property "Footprint" "Z_Custom_Footprints:CONN_1935776_PXC"
 			(at 100.33 83.82 0)
 			(effects
@@
 			)
 		)
-		(property "Footprint" "MountingHole:MountingHole_2.7mm_M2.5_DIN965_Pad"
+		(property "Footprint" "MountingHole:MountingHole_3.5mm_Pad"
 			(at 64.77 114.3 0)
 			(effects
@@
 			)
 		)
-		(property "Footprint" "MountingHole:MountingHole_2.7mm_M2.5_DIN965_Pad"
+		(property "Footprint" "MountingHole:MountingHole_3.5mm_Pad"
 			(at 64.77 121.92 0)
 			(effects
@@
 			)
 		)
-		(property "Footprint" "Potentiometer_THT:Potentiometer_ACP_CA9-V10_Vertical"
+		(property "Footprint" "Z_Custom_Footprints:POT_3362P"
 			(at 110.49 41.402 90)
 			(effects
@@
 			)
 		)
-		(property "Footprint" "Resistor_THT:R_Axial_DIN0204_L3.6mm_D1.6mm_P5.08mm_Horizontal"
+		(property "Footprint" "Resistor_THT:R_Axial_DIN0207_L6.3mm_D2.5mm_P10.16mm_Horizontal"
 			(at 165.862 69.85 90)
 			(effects
@@
 			)
 		)
-		(property "Footprint" "MountingHole:MountingHole_2.7mm_M2.5_DIN965_Pad"
+		(property "Footprint" "MountingHole:MountingHole_3.5mm_Pad"
 			(at 64.77 135.89 0)
 			(effects
@@
 			)
 		)
-		(property "Footprint" "Capacitor_THT:CP_Radial_D4.0mm_P1.50mm"
+		(property "Footprint" "Capacitor_THT:C_Disc_D3.0mm_W1.6mm_P2.50mm"
 			(at 143.2052 135.89 0)
 			(effects
@@
 			)
 		)
-		(property "Footprint" "Resistor_THT:R_Axial_DIN0204_L3.6mm_D1.6mm_P5.08mm_Horizontal"
+		(property "Footprint" "Resistor_THT:R_Axial_DIN0207_L6.3mm_D2.5mm_P10.16mm_Horizontal"
 			(at 110.49 39.878 90)
 			(effects
@@
 			)
 		)
-		(property "Footprint" "MountingHole:MountingHole_2.7mm_M2.5_DIN965_Pad"
+		(property "Footprint" "MountingHole:MountingHole_3.5mm_Pad"
 			(at 64.77 129.54 0)
 			(effects
@@
 			)
 		)
-		(property "Footprint" "Capacitor_THT:CP_Radial_D4.0mm_P1.50mm"
+		(property "Footprint" "Capacitor_THT:C_Disc_D3.0mm_W1.6mm_P2.50mm"
 			(at 143.2052 31.75 0)
 			(effects
@@
 			)
 		)
-		(property "Footprint" "Resistor_THT:R_Axial_DIN0204_L3.6mm_D1.6mm_P5.08mm_Horizontal"
+		(property "Footprint" "Resistor_THT:R_Axial_DIN0207_L6.3mm_D2.5mm_P10.16mm_Horizontal"
 			(at 110.49 127.762 90)
 			(effects
@@
 			)
 		)
-		(property "Footprint" "Capacitor_THT:CP_Radial_D4.0mm_P1.50mm"
+		(property "Footprint" "Capacitor_THT:C_Disc_D4.3mm_W1.9mm_P5.00mm"
 			(at 97.79 63.1952 0)
 			(effects
@@
 			)
 		)
-		(property "Footprint" "Resistor_THT:R_Axial_DIN0204_L3.6mm_D1.6mm_P5.08mm_Horizontal"
+		(property "Footprint" "Resistor_THT:R_Axial_DIN0207_L6.3mm_D2.5mm_P10.16mm_Horizontal"
 			(at 155.702 132.08 90)
 			(effects
@@
 			)
 		)
-		(property "Value" "Speaker Terminals"
+		(property "Value" "Speaker"
 			(at 210.82 86.3599 0)
 			(effects
@@
 			)
 		)
-		(property "Footprint" "Connector_Wire:SolderWire-2.5sqmm_1x02_P7.2mm_D2.4mm_OD3.6mm"
+		(property "Footprint" "Z_Custom_Footprints:CONN_1935776_PXC"
 			(at 208.28 83.82 0)
 			(effects
@@
 			)
 		)
-		(property "Footprint" "Resistor_THT:R_Axial_DIN0204_L3.6mm_D1.6mm_P5.08mm_Horizontal"
+		(property "Footprint" "Resistor_THT:R_Axial_DIN0207_L6.3mm_D2.5mm_P10.16mm_Horizontal"
 			(at 142.24 80.518 90)
 			(effects
@@
 			)
 		)
-		(property "Footprint" "Resistor_THT:R_Axial_DIN0204_L3.6mm_D1.6mm_P5.08mm_Horizontal"
+		(property "Footprint" "Resistor_THT:R_Axial_DIN0207_L6.3mm_D2.5mm_P10.16mm_Horizontal"
 			(at 165.862 97.79 90)
 			(effects
@@
 			)
 		)
-		(property "Footprint" "Resistor_THT:R_Axial_DIN0204_L3.6mm_D1.6mm_P5.08mm_Horizontal"
+		(property "Footprint" "Resistor_THT:R_Axial_DIN0207_L6.3mm_D2.5mm_P10.16mm_Horizontal"
 			(at 125.222 87.63 90)
 			(effects

Commit message: All footprints verified
Parts:
- C1, C7: footprint Capacitor_THT:CP_Radial_D4.0mm_P1.50mm -> Capacitor_THT:C_Rect_L7.0mm_W3.5mm_P5.00mm
- C3, C5: footprint Capacitor_THT:C_Disc_D4.3mm_W1.9mm_P5.00mm -> Capacitor_THT:CP_Radial_D5.0mm_P2.00mm
- C4, C6: footprint Capacitor_THT:C_Disc_D3.0mm_W1.6mm_P2.50mm -> Capacitor_THT:C_Disc_D5.1mm_W3.2mm_P5.00mm
- J1, J2, J3: footprint Z_Custom_Footprints:CONN_1935776_PXC -> Custom_Footprints:CONN_1935776_PXC
- R11, R7: footprint Z_Custom_Footprints:POT_3362P -> Custom_Footprints:POT_3362P
Changed lines of the file:
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@@
 			)
 		)
-		(property "Footprint" "Capacitor_THT:CP_Radial_D4.0mm_P1.50mm"
+		(property "Footprint" "Capacitor_THT:C_Rect_L7.0mm_W3.5mm_P5.00mm"
 			(at 186.3852 73.66 0)
 			(effects
@@
 		)
 		(instances
-			(project "Dorr_Amp_Draft3"
+			(project "Dorr_Amp_REV-"
 				(path "/cc9ff92f-9b14-4efc-8fda-45ee1c134506"
 					(reference "C7")
@@
 		)
 		(instances
-			(project "Dorr_Amp_Draft3"
+			(project "Dorr_Amp_REV-"
 				(path "/cc9ff92f-9b14-4efc-8fda-45ee1c134506"
 					(reference "R18")
@@
 		)
 		(instances
-			(project "Dorr_Amp_Draft3"
+			(project "Dorr_Amp_REV-"
 				(path "/cc9ff92f-9b14-4efc-8fda-45ee1c134506"
 					(reference "R14")
@@
 		)
 		(instances
-			(project "Dorr_Amp_Draft3"
+			(project "Dorr_Amp_REV-"
 				(path "/cc9ff92f-9b14-4efc-8fda-45ee1c134506"
 					(reference "#PWR05")
@@
 		)
 		(instances
-			(project "Dorr_Amp_Draft3"
+			(project "Dorr_Amp_REV-"
 				(path "/cc9ff92f-9b14-4efc-8fda-45ee1c134506"
 					(reference "R2")
@@
 		)
 		(instances
-			(project "Dorr_Amp_Draft3"
+			(project "Dorr_Amp_REV-"
 				(path "/cc9ff92f-9b14-4efc-8fda-45ee1c134506"
 					(reference "R6")
@@
 		)
 		(instances
-			(project "Dorr_Amp_Draft3"
+			(project "Dorr_Amp_REV-"
 				(path "/cc9ff92f-9b14-4efc-8fda-45ee1c134506"
 					(reference "#PWR06")
@@
 		)
 		(instances
-			(project "Dorr_Amp_Draft3"
+			(project "Dorr_Amp_REV-"
 				(path "/cc9ff92f-9b14-4efc-8fda-45ee1c134506"
 					(reference "C8")
@@
 		)
 		(instances
-			(project "Dorr_Amp_Draft3"
+			(project "Dorr_Amp_REV-"
 				(path "/cc9ff92f-9b14-4efc-8fda-45ee1c134506"
 					(reference "R5")
@@
 			)
 		)
-		(property "Footprint" "Capacitor_THT:C_Disc_D4.3mm_W1.9mm_P5.00mm"
+		(property "Footprint" "Capacitor_THT:CP_Radial_D5.0mm_P2.00mm"
 			(at 97.79 104.4448 0)
 			(effects
@@
 		)
 		(instances
-			(project "Dorr_Amp_Draft3"
+			(project "Dorr_Amp_REV-"
 				(path "/cc9ff92f-9b14-4efc-8fda-45ee1c134506"
 					(reference "C3")
@@
 		)
 		(instances
-			(project "Dorr_Amp_Draft3"
+			(project "Dorr_Amp_REV-"
 				(path "/cc9ff92f-9b14-4efc-8fda-45ee1c134506"
 					(reference "TP2")
@@
 		)
 		(instances
-			(project "Dorr_Amp_Draft3"
+			(project "Dorr_Amp_REV-"
 				(path "/cc9ff92f-9b14-4efc-8fda-45ee1c134506"
 					(reference "TP1")
@@
 		)
 		(instances
-			(project "Dorr_Amp_Draft3"
+			(project "Dorr_Amp_REV-"
 				(path "/cc9ff92f-9b14-4efc-8fda-45ee1c134506"
 					(reference "D4")
@@
 			)
 		)
-		(property "Footprint" "Z_Custom_Footprints:POT_3362P"
+		(property "Footprint" "Custom_Footprints:POT_3362P"
 			(at 110.49 126.238 90)
 			(effects
@@
 		)
 		(instances
-			(project "Dorr_Amp_Draft3"
+			(project "Dorr_Amp_REV-"
 				(path "/cc9ff92f-9b14-4efc-8fda-45ee1c134506"
 					(reference "R7")
@@
 		)
 		(instances
-			(project "Dorr_Amp_Draft3"
+			(project "Dorr_Amp_REV-"
 				(path "/cc9ff92f-9b14-4efc-8fda-45ee1c134506"
 					(reference "R13")
@@
 		)
 		(instances
-			(project "Dorr_Amp_Draft3"
+			(project "Dorr_Amp_REV-"
 				(path "/cc9ff92f-9b14-4efc-8fda-45ee1c134506"
 					(reference "R10")
@@
 			)
 		)
-		(property "Footprint" "Capacitor_THT:CP_Radial_D4.0mm_P1.50mm"
+		(property "Footprint" "Capacitor_THT:C_Rect_L7.0mm_W3.5mm_P5.00mm"
 			(at 186.3852 93.98 0)
 			(effects
@@
 		)
 		(instances
-			(project "Dorr_Amp_Draft3"
+			(project "Dorr_Amp_REV-"
 				(path "/cc9ff92f-9b14-4efc-8fda-45ee1c134506"
 					(reference "C1")
@@
 		)
 		(instances
-			(project "Dorr_Amp_Draft3"
+			(project "Dorr_Amp_REV-"
 				(path "/cc9ff92f-9b14-4efc-8fda-45ee1c134506"
 					(reference "R16")
@@
 		)
 		(instances
-			(project "Dorr_Amp_Draft3"
+			(project "Dorr_Amp_REV-"
 				(path "/cc9ff92f-9b14-4efc-8fda-45ee1c134506"
 					(reference "Q10")
@@
 		)
 		(instances
-			(project "Dorr_Amp_Draft3"
+			(project "Dorr_Amp_REV-"
 				(path "/cc9ff92f-9b14-4efc-8fda-45ee1c134506"
 					(reference "#PWR07")
@@
 			)
 		)
-		(property "Footprint" "Z_Custom_Footprints:CONN_1935776_PXC"
+		(property "Footprint" "Custom_Footprints:CONN_1935776_PXC"
 			(at 83.82 83.82 0)
 			(effects
@@
 		)
 		(instances
-			(project "Dorr_Amp_Draft3"
+			(project "Dorr_Amp_REV-"
 				(path "/cc9ff92f-9b14-4efc-8fda-45ee1c134506"
 					(reference "J2")
@@
 		)
 		(instances
-			(project "Dorr_Amp_Draft3"
+			(project "Dorr_Amp_REV-"
 				(path "/cc9ff92f-9b14-4efc-8fda-45ee1c134506"
 					(reference "R4")
@@
 			)
 		)
-		(property "Footprint" "Z_Custom_Footprints:CONN_1935776_PXC"
+		(property "Footprint" "Custom_Footprints:CONN_1935776_PXC"
 			(at 100.33 83.82 0)
 			(effects
@@
 		)
 		(instances
-			(project "Dorr_Amp_Draft3"
+			(project "Dorr_Amp_REV-"
 				(path "/cc9ff92f-9b14-4efc-8fda-45ee1c134506"
 					(reference "J3")
@@
 		)
 		(instances
-			(project "Dorr_Amp_Draft3"
+			(project "Dorr_Amp_REV-"
 				(path "/cc9ff92f-9b14-4efc-8fda-45ee1c134506"
 					(reference "#PWR01")
@@
 			)
 		)
-		(property "Footprint" "Z_Custom_Footprints:POT_3362P"
+		(property "Footprint" "Custom_Footprints:POT_3362P"
 			(at 110.49 41.402 90)
 			(effects
@@
 		)
 		(instances
-			(project "Dorr_Amp_Draft3"
+			(project "Dorr_Amp_REV-"
 				(path "/cc9ff92f-9b14-4efc-8fda-45ee1c134506"
 					(reference "R11")
@@
 		)
 		(instances
-			(project "Dorr_Amp_Draft3"
+			(project "Dorr_Amp_REV-"
 				(path "/cc9ff92f-9b14-4efc-8fda-45ee1c134506"
 					(reference "R17")
@@
 		)
 		(instances
-			(project ""
+			(project "Dorr_Amp_REV-"
 				(path "/cc9ff92f-9b14-4efc-8fda-45ee1c134506"
 					(reference "#PWR09")
@@
 			)
 		)
-		(property "Footprint" "Capacitor_THT:C_Disc_D3.0mm_W1.6mm_P2.50mm"
+		(property "Footprint" "Capacitor_THT:C_Disc_D5.1mm_W3.2mm_P5.00mm"
 			(at 143.2052 135.89 0)
 			(effects
@@
 		)
 		(instances
-			(project "Dorr_Amp_Draft3"
+			(project "Dorr_Amp_REV-"
 				(path "/cc9ff92f-9b14-4efc-8fda-45ee1c134506"
 					(reference "C4")
@@
 		)
 		(instances
-			(project "Dorr_Amp_Draft3"
+			(project "Dorr_Amp_REV-"
 				(path "/cc9ff92f-9b14-4efc-8fda-45ee1c134506"
 					(reference "#PWR02")
@@
 		)
 		(instances
-			(project "Dorr_Amp_Draft3"
+			(project "Dorr_Amp_REV-"
 				(path "/cc9ff92f-9b14-4efc-8fda-45ee1c134506"
 					(reference "#FLG01")
@@
 		)
 		(instances
-			(project "Dorr_Amp_Draft3"
+			(project "Dorr_Amp_REV-"
 				(path "/cc9ff92f-9b14-4efc-8fda-45ee1c134506"
 					(reference "D3")
@@
 		)
 		(instances
-			(project "Dorr_Amp_Draft3"
+			(project "Dorr_Amp_REV-"
 				(path "/cc9ff92f-9b14-4efc-8fda-45ee1c134506"
 					(reference "Q3")
@@
 		)
 		(instances
-			(project "Dorr_Amp_Draft3"
+			(project "Dorr_Amp_REV-"
 				(path "/cc9ff92f-9b14-4efc-8fda-45ee1c134506"
 					(reference "R12")
@@
 		)
 		(instances
-			(project "Dorr_Amp_Draft3"
+			(project "Dorr_Amp_REV-"
 				(path "/cc9ff92f-9b14-4efc-8fda-45ee1c134506"
 					(reference "Q1")
@@
 			)
 		)
-		(property "Footprint" "Capacitor_THT:C_Disc_D3.0mm_W1.6mm_P2.50mm"
+		(property "Footprint" "Capacitor_THT:C_Disc_D5.1mm_W3.2mm_P5.00mm"
 			(at 143.2052 31.75 0)
 			(effects
@@
 		)
 		(instances
-			(project "Dorr_Amp_Draft3"
+			(project "Dorr_Amp_REV-"
 				(path "/cc9ff92f-9b14-4efc-8fda-45ee1c134506"
 					(reference "C6")
@@
 		)
 		(instances
-			(project "Dorr_Amp_Draft3"
+			(project "Dorr_Amp_REV-"
 				(path "/cc9ff92f-9b14-4efc-8fda-45ee1c134506"
 					(reference "R8")
@@
 		)
 		(instances
-			(project "Dorr_Amp_Draft3"
+			(project "Dorr_Amp_REV-"
 				(path "/cc9ff92f-9b14-4efc-8fda-45ee1c134506"
 					(reference "Q4")
@@
 			)
 		)
-		(property "Footprint" "Capacitor_THT:C_Disc_D4.3mm_W1.9mm_P5.00mm"
+		(property "Footprint" "Capacitor_THT:CP_Radial_D5.0mm_P2.00mm"
 			(at 97.79 63.1952 0)
 			(effects
@@
 		)
 		(instances
-			(project "Dorr_Amp_Draft3"
+			(project "Dorr_Amp_REV-"
 				(path "/cc9ff92f-9b14-4efc-8fda-45ee1c134506"
 					(reference "C5")
@@
 		)
 		(instances
-			(project "Dorr_Amp_Draft3"
+			(project "Dorr_Amp_REV-"
 				(path "/cc9ff92f-9b14-4efc-8fda-45ee1c134506"
 					(reference "R9")
@@
 		)
 		(instances
-			(project "Dorr_Amp_Draft3"
+			(project "Dorr_Amp_REV-"
 				(path "/cc9ff92f-9b14-4efc-8fda-45ee1c134506"
 					(reference "Q8")
@@
 		)
 		(instances
-			(project "Dorr_Amp_Draft3"
+			(project "Dorr_Amp_REV-"
 				(path "/cc9ff92f-9b14-4efc-8fda-45ee1c134506"
 					(reference "Q7")
@@
 			)
 		)
-		(property "Footprint" "Z_Custom_Footprints:CONN_1935776_PXC"
+		(property "Footprint" "Custom_Footprints:CONN_1935776_PXC"
 			(at 208.28 83.82 0)
 			(effects
@@
 		)
 		(instances
-			(project "Dorr_Amp_Draft3"
+			(project "Dorr_Amp_REV-"
 				(path "/cc9ff92f-9b14-4efc-8fda-45ee1c134506"
 					(reference "J1")
@@
 		)
 		(instances
-			(project "Dorr_Amp_Draft3"
+			(project "Dorr_Amp_REV-"
 				(path "/cc9ff92f-9b14-4efc-8fda-45ee1c134506"
 					(reference "#PWR04")
@@
 		)
 		(instances
-			(project "Dorr_Amp_Draft3"
+			(project "Dorr_Amp_REV-"
 				(path "/cc9ff92f-9b14-4efc-8fda-45ee1c134506"
 					(reference "R15")
@@
 		)
 		(instances
-			(project "Dorr_Amp_Draft3"
+			(project "Dorr_Amp_REV-"
 				(path "/cc9ff92f-9b14-4efc-8fda-45ee1c134506"
 					(reference "D2")
@@
 		)
 		(instances
-			(project "Dorr_Amp_Draft3"
+			(project "Dorr_Amp_REV-"
 				(path "/cc9ff92f-9b14-4efc-8fda-45ee1c134506"
 					(reference "R3")
@@
 		)
 		(instances
-			(project "Dorr_Amp_Draft3"
+			(project "Dorr_Amp_REV-"
 				(path "/cc9ff92f-9b14-4efc-8fda-45ee1c134506"
 					(reference "D1")
@@
 		)
 		(instances
-			(project "Dorr_Amp_Draft3"
+			(project "Dorr_Amp_REV-"
 				(path "/cc9ff92f-9b14-4efc-8fda-45ee1c134506"
 					(reference "R1")
@@
 		)
 		(instances
-			(project "Dorr_Amp_Draft3"
+			(project "Dorr_Amp_REV-"
 				(path "/cc9ff92f-9b14-4efc-8fda-45ee1c134506"
 					(reference "Q6")
@@
 		)
 		(instances
-			(project "Dorr_Amp_Draft3"
+			(project "Dorr_Amp_REV-"
 				(path "/cc9ff92f-9b14-4efc-8fda-45ee1c134506"
 					(reference "Q2")
@@
 		)
 		(instances
-			(project "Dorr_Amp_Draft3"
+			(project "Dorr_Amp_REV-"
 				(path "/cc9ff92f-9b14-4efc-8fda-45ee1c134506"
 					(reference "#PWR03")
