File: docs/Kicad Files/Amplifier/Amplifier/Amplifier, REV-/Dorr_Amp_REV-.kicad_pcb (KiCad board)
At the start: 2 copper layers, 152.7 x 76.2 mm, 48 parts, among them J1 Speaker, J2 Input Terminals, J3 Power Input, Q1 2N3904, Q10 QD44H8G, Q2 QD45H8G, Q3 2N3904, Q4 2N3906, Q5 QD44H8G, Q6 2N3904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

Commit message: PCB traces updated - waiting feedback from Mark
Parts:
- moved R7 14.7 mm to (73.2, 119.8), turned to 90 degrees
- moved Q4 3.53 mm to (116.7, 120.9), turned to 90 degrees
- moved C6 3.50 mm to (107.6, 69.7)
Routing:
- net Net-(Q10-C): track 45.1 -> 62.5 mm
- net Net-(D1-K): track 69.9 -> 57.0 mm
- net Net-(Q10-B): track 52.9 -> 46.2 mm
- net /18V: track 121.1 -> 126.0 mm
- net Net-(Q4-E): track 61.7 -> 65.7 mm
- net Net-(D4-K): track 43.2 -> 46.1 mm
- net GND: track 2.78 -> 0.00 mm, vias 0 -> 6
- net Net-(Q1-E): track 65.6 -> 63.3 mm
- net Net-(Q2-C): track 63.3 -> 61.2 mm
- net Net-(D2-K): track 30.9 -> 32.6 mm
- net Net-(Q2-B): track 41.8 -> 43.1 mm
- net Net-(Q4-C): track 38.9 -> 38.0 mm
