File: docs/Kicad Files/Amplifier/Archive/Amplifier, REV-/Dorr_Amp_REV-.kicad_pcb (KiCad board)
At the start: 2 copper layers, 152.7 x 76.2 mm, 48 parts, among them J1 Speaker, J2 Input Terminals, J3 Power Input, Q1 2N3904, Q10 QD44H8G, Q2 QD45H8G, Q3 2N3904, Q4 2N3906, Q5 QD44H8G, Q6 2N3904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

Commit message: cleaned up amp directory
Parts:
- moved R7 14.7 mm to (58.6, 117.9), turned to 0 degrees
- moved R13 5.33 mm to (92.9, 101.0)
- moved Q4 3.53 mm to (114.7, 118.0), turned to -90 degrees
- moved C6 3.50 mm to (109.6, 72.6)
- moved J1 3.35 mm to (181.0, 98.4)
- moved Q8 2.25 mm to (114.7, 87.4), turned to 90 degrees
- moved R2 1.69 mm to (137.7, 113.3)
- moved H2 1.20 mm to (187.4, 66.3)
- moved H3 1.17 mm to (42.0, 134.8)
- moved H1 0.94 mm to (42.3, 66.7)
- moved H4 0.88 mm to (187.3, 134.8)
- moved C3 0.72 mm to (44.9, 128.3)
- moved Q1 0.64 mm to (114.7, 110.3)
- moved Q7 0.54 mm to (111.0, 93.2)
Routing:
- net Net-(Q4-E): track 65.7 -> 0.00 mm
- net Net-(J1-Pin_2): track 93.8 -> 29.9 mm
- net Net-(Q1-E): track 63.3 -> 0.00 mm
- net Net-(Q10-C): track 62.5 -> 0.00 mm
- net Net-(Q2-C): track 61.2 -> 0.00 mm
- net Net-(D3-K): track 60.2 -> 0.00 mm
- net Net-(C8-Pad1): track 67.2 -> 8.17 mm
- net Net-(D1-K): track 57.0 -> 0.00 mm
- net Net-(Q10-B): track 46.2 -> 0.00 mm
- net Net-(D4-K): track 46.1 -> 0.00 mm
- net Net-(Q2-B): track 43.1 -> 0.00 mm
- net Net-(Q1-C): track 41.3 -> 0.00 mm
- net Net-(J2-Pin_2): track 40.5 -> 0.00 mm
- net Net-(Q4-C): track 38.0 -> 0.00 mm
- net Net-(D1-A): track 34.9 -> 0.00 mm
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