File: docs/Kicad Files/Amplifier/Power_Amp_RevA/Power_Amp_RevA.kicad_pcb (KiCad board)
At the start: 2 copper layers, 152.7 x 76.2 mm, 48 parts, among them J1 Speaker, J2 Input Terminals, J3 Power Input, Q1 2N3904, Q10 QD44H8G, Q2 QD45H8G, Q3 2N3904, Q4 2N3906, Q5 QD44H8G, Q6 2N3904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

Commit message: changed some footprints per Mark
-routed input traces to back of PCB
-changed footprints of pots and terminal blocks
-flipped terminal blocks so orientation is correct
-added terminal block descriptions
Parts:
- J1, J2, J3: footprint Z_Custom_Footprints:CONN_1935776_PXC -> TerminalBlock_Phoenix:TerminalBlock_Phoenix_MKDS-1,5-2_1x02_P5.00mm_Horizontal
- RV1, RV2: footprint Z_Custom_Footprints:POT_3362P -> Potentiometer_THT:Potentiometer_Bourns_3386P_Vertical
- moved J3 31.5 mm to (49.0, 89.3), turned to -90 degrees
- moved J1 6.16 mm to (174.8, 103.9), turned to 90 degrees
- moved RV2 3.53 mm to (72.8, 116.2)
- moved C3 2.20 mm to (49.1, 130.3)
- moved J2 2.14 mm to (49.1, 118.2), turned to -90 degrees
- moved R10 1.66 mm to (62.1, 82.3)
Connections:
- C8 pad 2: Net-(J1-Pin_1) -> Net-(J1-Pin_2)
- R3 pad 2: Net-(J1-Pin_2) -> Net-(J1-Pin_1)
- R4 pad 1: Net-(J1-Pin_2) -> Net-(J1-Pin_1)
- R5 pad 1: Net-(J1-Pin_2) -> Net-(J1-Pin_1)
- TP1 pad 1: Net-(J1-Pin_2) -> Net-(J1-Pin_1)
Routing:
- net Net-(J1-Pin_2): track 93.8 -> 19.1 mm
- net Net-(J1-Pin_1): track 19.8 -> 92.2 mm
- net /18V: track 126.0 -> 159.8 mm
- net Net-(J2-Pin_2): track 40.5 -> 62.3 mm
- net Net-(D1-K): track 53.2 -> 57.9 mm
- net Net-(D3-K): track 57.4 -> 58.4 mm
- net Net-(J2-Pin_1): track 14.4 -> 15.0 mm
Other:
- board text added: "18V + -"
- board text added: "Input"
- board text added: "Speaker (8 Ohms)"
