File: docs/Kicad Files/Amplifier/Power_Amp_RevB/Power_Amp_RevB.kicad_sch (KiCad schematic)
At the start: 48 parts, among them J1 Speaker, J2 Input Terminals, J3 Power Input, Q1 2N3904, Q10 QD44H8G, Q2 QD45H8G, Q3 2N3904, Q4 2N3906, Q5 QD44H8G, Q6 2N3904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

Commit message: final changes to both PCBs before review
Parts:
- TP1, TP2: footprint TestPoint:TestPoint_Plated_Hole_D2.0mm -> TestPoint:TestPoint_THTPad_D2.0mm_Drill1.0mm
Changed lines of the file:
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@@
 			)
 		)
-		(property "Footprint" "TestPoint:TestPoint_Plated_Hole_D2.0mm"
+		(property "Footprint" "TestPoint:TestPoint_THTPad_D2.0mm_Drill1.0mm"
 			(at 184.15 62.23 0)
 			(effects
@@
 			)
 		)
-		(property "Footprint" "TestPoint:TestPoint_Plated_Hole_D2.0mm"
+		(property "Footprint" "TestPoint:TestPoint_THTPad_D2.0mm_Drill1.0mm"
 			(at 184.15 105.41 0)
 			(effects
