File: docs/Kicad Files/Atmega_BM83_Board/Atmega_BM83.kicad_pcb (KiCad board)
At the start: 2 copper layers, 114.3 x 88.9 mm, 35 parts, among them J1 18V, J10 ICE Header, J2 Out to Amp, J3 PWR SW, J4 Volume POT, J5 Pairing BTN, J6 PWR LED, J7 Pair LED, J8 Conn_01x12, J9 Conn_01x12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

Commit message: widened traces per Mark's suggestion. connected  AVCC and C7 as per datasheet.
Parts:
- moved C7 7.06 mm to (145.3, 91.8), turned to 0 degrees
Connections:
- C7 pad 1: GND -> 5V
- C7 pad 2: Net-(U3-AVCC) -> GND
- U3 pad 20: Net-(U3-AVCC) -> 5V
Routing:
- net Net-(U3-AVCC): track 61.5 -> 0.00 mm, vias 1 -> 0
- net 5V: track 166.7 -> 205.2 mm
- net MOSI: track 22.6 -> 21.5 mm
- net 8V: track 82.6 -> 83.2 mm
- net Net-(C3-Pad2): track 23.4 -> 22.9 mm
- net GND: vias 8 -> 10
