File: docs/Kicad Files/Power Distribution Jack/PD Jack/PD Jack.kicad_pcb (KiCad board)
At the start: 2 copper layers, 69.8 x 71.1 mm, 8 parts, among them J1 Barrel_Jack_Switch_MountingPin, J2(+)1 Screw_Terminal_01x03, J3(-)1 Screw_Terminal_01x03

Commit message: New Updates to PD Jack
Parts:
- added H3: MountingHole_Pad, MountingHole:MountingHole_3.5mm_Pad, F.Cu at (108.0, 72.4)
- added H4: MountingHole_Pad, MountingHole:MountingHole_3.5mm_Pad, F.Cu at (108.0, 130.8)
- renumbered J2(+)1 to J2(+), J3(-)1 to J3(-)
Routing:
- net Net-(J3(-)1-Pin_1): track 63.5 -> 109.1 mm
- net 18V: track 60.1 -> 85.4 mm
Other:
- board text added: "SAN DIEGO STATE UNIVERSITY COLLEGE OF ENGINEERING DEPARTMENT OF ELECTRICAL & COMPUTER ENGINEERING TEAM BOOM: POWER DISTRIBUTION JACK, REV. A"
