File: docs/Kicad Files/Power Distribution Jack/PD Jack/PD Jack.kicad_sch (KiCad schematic)
At the start: 8 parts, among them J1 Barrel_Jack_Switch_MountingPin, J2(+)1 Screw_Terminal_01x03, J3(-)1 Screw_Terminal_01x03

Commit message: New Updates to PD Jack
Parts:
- added H3, H4: MountingHole_Pad, MountingHole:MountingHole_3.5mm_Pad, symbol Mechanical:MountingHole_Pad
Connections:
- net GND: now also H3.1, H4.1
Other:
- moved on the sheet: H2
