File: docs/Kicad Files/Power Distribution Jack/PD Jack/PD Jack_RevA.kicad_pcb (KiCad board)
At the start: 2 copper layers, 69.8 x 71.1 mm, 10 parts, among them J1 Barrel_Jack_Switch_MountingPin, J2(+) Screw_Terminal_01x03, J3(-) Screw_Terminal_01x03

Commit message: PD Jack_RevA
Parts:
- removed J3(-): Screw_Terminal_01x03, TerminalBlock_Phoenix:TerminalBlock_Phoenix_MKDS-1,5-3_1x03_P5.00mm_Horizontal
- added (-)J3: Screw_Terminal_01x03, TerminalBlock_Phoenix:TerminalBlock_Phoenix_MKDS-1,5-3_1x03_P5.00mm_Horizontal, F.Cu at (164.1, 118.0)
- moved H3 16.5 mm to (124.5, 72.4)
- moved H4 16.5 mm to (124.5, 130.8)
- moved J1 13.8 mm to (134.3, 99.4)
- moved (+)J2 9.92 mm to (163.8, 99.0), turned to 90 degrees
- moved D1 4.90 mm to (124.9, 80.2)
- moved H1 1.09 mm to (165.1, 72.6)
- moved H2 1.09 mm to (165.1, 131.0)
- renumbered J2(+) to (+)J2
Connections:
- J1 pad 2: Net-(J3(-)1-Pin_1) -> GND
- J1 pad 3: Net-(J3(-)1-Pin_1) -> GND
Routing:
- net Net-(J3(-)1-Pin_1): track 109.1 -> 0.00 mm
- net GND: track 47.2 -> 143.7 mm
- net 18V: track 85.4 -> 69.5 mm
- net Net-(D1-A): track 21.5 -> 18.9 mm
Other:
- board size 69.8 x 71.1 mm -> 50.8 x 71.1 mm
- board text added: "SAN DIEGO STATE UNIVERSITY COLLEGE OF ENGINEERING ELECTRICAL & COMPUTER ENGINEERING TEAM BOOM POWER DISTRIBUTION JACK, REV. A"
- board text removed: "SAN DIEGO STATE UNIVERSITY COLLEGE OF ENGINEERING DEPARTMENT OF ELECTRICAL & COMPUTER ENGINEERING TEAM BOOM: POWER DISTRIBUTION JACK, REV. A"
